Commit message: modifed car model

File: racecar_description/urdf/racecar.xacro (robot description, xacro)
@@ -26,4 +26,5 @@
   </joint>
   <!-- Add the left rear wheel with its joints and tranmissions -->
+  <!--
   <link name="left_rear_wheel">
     <inertial>
@@ -46,5 +47,7 @@
   </joint>
   <xacro:wheel_transmission name="left_rear_wheel" />
+  -->
   <!-- Add the right rear wheel with its joints and tranmissions -->
+  <!--
   <link name="right_rear_wheel">
     <inertial>
@@ -67,4 +70,5 @@
   </joint>
   <xacro:wheel_transmission name="right_rear_wheel" />
+  -->
   <!-- Add the left steering hinge with its joints and tranmissions -->
   <link name="left_steering_hinge">
@@ -104,4 +108,5 @@
   <xacro:steering_hinge_transmission name="right_steering_hinge" />
   <!-- Add the left front wheel with its joints and tranmissions -->
+  <!--
   <link name="left_front_wheel">
     <inertial>
@@ -124,5 +129,7 @@
   </joint>
   <xacro:wheel_transmission name="left_front_wheel" />
+  -->
   <!-- Add the left front wheel with its joints and tranmissions -->
+  <!--
   <link name="right_front_wheel">
     <inertial>
@@ -145,4 +152,5 @@
   </joint>
   <xacro:wheel_transmission name="right_front_wheel" />
+  -->
   <!-- Add Hokuyo laser scanner -->
   <link name="laser">
@@ -165,5 +173,5 @@
   </link>
   <joint name="hokuyo_joint" type="fixed">
-    <origin xyz="0.265 0.0 0.075" rpy="0 0 0"/>
+    <origin xyz="0.265 0.0 0.075" rpy="0 -0.05 0"/>
     <parent link="chassis" />
     <child link="laser" />

Commit message: Change urdf to use full circle laser scan

File: racecar_description/urdf/racecar.xacro (robot description, xacro)
@@ -173,5 +173,5 @@
   </link>
   <joint name="hokuyo_joint" type="fixed">
-    <origin xyz="0.265 0.0 0.075" rpy="0 -0.05 0"/>
+    <origin xyz="0.265 0.0 0.075" rpy="0 0 0"/>
     <parent link="chassis" />
     <child link="laser" />

Commit message: Set laser scan to not detect other cars

File: racecar_description/urdf/racecar.xacro (robot description, xacro)
@@ -166,7 +166,10 @@
     <visual>
       <origin xyz="0 0 0" rpy="0 0 0"/>
-      <geometry>
+      <transparency>1</transparency>
+      <geometry>
+        <!--
         <mesh filename="package://racecar_description/meshes/hokuyo.dae"/>
-        <material name="grey" />
+        -->
+        <material>Gazebo/GreyTransparent</material>
       </geometry>
     </visual>

Commit message: Revert "modifed car model"
This reverts commit 931a386a9db19e2917b7970a1897e9215a24f032.

File: racecar_description/urdf/racecar.xacro (robot description, xacro)
@@ -26,5 +26,4 @@
   </joint>
   <!-- Add the left rear wheel with its joints and tranmissions -->
-  <!--
   <link name="left_rear_wheel">
     <inertial>
@@ -47,7 +46,5 @@
   </joint>
   <xacro:wheel_transmission name="left_rear_wheel" />
-  -->
   <!-- Add the right rear wheel with its joints and tranmissions -->
-  <!--
   <link name="right_rear_wheel">
     <inertial>
@@ -70,5 +67,4 @@
   </joint>
   <xacro:wheel_transmission name="right_rear_wheel" />
-  -->
   <!-- Add the left steering hinge with its joints and tranmissions -->
   <link name="left_steering_hinge">
@@ -108,5 +104,4 @@
   <xacro:steering_hinge_transmission name="right_steering_hinge" />
   <!-- Add the left front wheel with its joints and tranmissions -->
-  <!--
   <link name="left_front_wheel">
     <inertial>
@@ -129,7 +124,5 @@
   </joint>
   <xacro:wheel_transmission name="left_front_wheel" />
-  -->
   <!-- Add the left front wheel with its joints and tranmissions -->
-  <!--
   <link name="right_front_wheel">
     <inertial>
@@ -152,5 +145,4 @@
   </joint>
   <xacro:wheel_transmission name="right_front_wheel" />
-  -->
   <!-- Add Hokuyo laser scanner -->
   <link name="laser">
@@ -166,10 +158,7 @@
     <visual>
       <origin xyz="0 0 0" rpy="0 0 0"/>
-      <transparency>1</transparency>
-      <geometry>
-        <!--
+      <geometry>
         <mesh filename="package://racecar_description/meshes/hokuyo.dae"/>
-        -->
-        <material>Gazebo/GreyTransparent</material>
+        <material name="grey" />
       </geometry>
     </visual>
